File: pcb_redesign/_autosave-pcb_redesign.kicad_sch (KiCad schematic)
At the start: 6 parts, among them U1 ESP32-S3-WROOM-1

Commit message: 12.21 may 11
Other:
- added sheet Connector (connector.kicad_sch)
Changed lines of the file:
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@@
   (junction (at 66.04 175.26) (diameter 0) (color 0 0 0 0)
   )
+  (junction (at 74.93 43.18) (diameter 0) (color 0 0 0 0)
+  )
+  (wire (pts (xy 189.23 91.44) (xy 199.39 91.44))
+    (stroke (width 0) (type default))
+  )
+  (wire (pts (xy 74.93 34.29) (xy 74.93 43.18))
+    (stroke (width 0) (type default))
+  )
   (wire (pts (xy 66.04 175.26) (xy 66.04 177.8))
     (stroke (width 0) (type default))
@@
     (stroke (width 0) (type default))
   )
+  (wire (pts (xy 189.23 129.54) (xy 199.39 129.54))
+    (stroke (width 0) (type default))
+  )
+  (wire (pts (xy 189.23 119.38) (xy 199.39 119.38))
+    (stroke (width 0) (type default))
+  )
+  (wire (pts (xy 189.23 99.06) (xy 199.39 99.06))
+    (stroke (width 0) (type default))
+  )
+  (wire (pts (xy 189.23 93.98) (xy 199.39 93.98))
+    (stroke (width 0) (type default))
+  )
+  (wire (pts (xy 189.23 106.68) (xy 199.39 106.68))
+    (stroke (width 0) (type default))
+  )
   (wire (pts (xy 88.9 78.74) (xy 97.79 78.74))
     (stroke (width 0) (type default))
@@
     (stroke (width 0) (type default))
   )
+  (wire (pts (xy 189.23 114.3) (xy 199.39 114.3))
+    (stroke (width 0) (type default))
+  )
   (wire (pts (xy 189.23 78.74) (xy 199.39 78.74))
     (stroke (width 0) (type default))
   )
-  (wire (pts (xy 67.31 43.18) (xy 143.51 43.18))
+  (wire (pts (xy 189.23 116.84) (xy 199.39 116.84))
+    (stroke (width 0) (type default))
+  )
+  (wire (pts (xy 189.23 88.9) (xy 199.39 88.9))
+    (stroke (width 0) (type default))
+  )
+  (wire (pts (xy 67.31 43.18) (xy 74.93 43.18))
     (stroke (width 0) (type default))
   )
@@
     (stroke (width 0) (type default))
   )
+  (wire (pts (xy 189.23 124.46) (xy 199.39 124.46))
+    (stroke (width 0) (type default))
+  )
   (wire (pts (xy 36.83 55.88) (xy 36.83 69.85))
     (stroke (width 0) (type default))
   )
+  (wire (pts (xy 189.23 111.76) (xy 199.39 111.76))
+    (stroke (width 0) (type default))
+  )
   (wire (pts (xy 66.04 172.72) (xy 66.04 175.26))
     (stroke (width 0) (type default))
@@
     (stroke (width 0) (type default))
   )
+  (wire (pts (xy 189.23 104.14) (xy 199.39 104.14))
+    (stroke (width 0) (type default))
+  )
   (wire (pts (xy 189.23 60.96) (xy 199.39 60.96))
     (stroke (width 0) (type default))
@@
     (stroke (width 0) (type default))
   )
+  (wire (pts (xy 189.23 109.22) (xy 199.39 109.22))
+    (stroke (width 0) (type default))
+  )
+  (wire (pts (xy 189.23 101.6) (xy 199.39 101.6))
+    (stroke (width 0) (type default))
+  )
+  (wire (pts (xy 74.93 43.18) (xy 143.51 43.18))
+    (stroke (width 0) (type default))
+  )
+  (wire (pts (xy 189.23 86.36) (xy 199.39 86.36))
+    (stroke (width 0) (type default))
+  )
   (wire (pts (xy 189.23 73.66) (xy 199.39 73.66))
     (stroke (width 0) (type default))
@@
     (stroke (width 0) (type default))
   )
+  (wire (pts (xy 189.23 96.52) (xy 199.39 96.52))
+    (stroke (width 0) (type default))
+  )
   (wire (pts (xy 88.9 124.46) (xy 97.79 124.46))
     (stroke (width 0) (type default))
   )
   (wire (pts (xy 189.23 58.42) (xy 199.39 58.42))
+    (stroke (width 0) (type default))
+  )
+  (wire (pts (xy 189.23 127) (xy 199.39 127))
+    (stroke (width 0) (type default))
+  )
+  (wire (pts (xy 189.23 121.92) (xy 199.39 121.92))
     (stroke (width 0) (type default))
   )
@@
     (effects (font (size 1.27 1.27)) (justify left bottom))
   )
-  (text "Have I used this label correctly??" (at 71.12 39.37 0)
+  (text "Have I used this label correctly??" (at 71.12 30.48 0)
     (effects (font (size 1.27 1.27)) (justify left bottom))
   )
@@
     )
   )
-  (netclass_flag "" (length 2.54) (shape round) (at 74.93 43.18 0) (fields_autoplaced)
-    (effects (font (size 1.27 1.27)) (justify left bottom))
-    (property "Netclass" "ESP32_3V3" (at 75.6285 40.64 0)
+  (netclass_flag "" (length 2.54) (shape round) (at 74.93 34.29 0) (fields_autoplaced)
+    (effects (font (size 1.27 1.27)) (justify left bottom))
+    (property "Netclass" "ESP32_3V3" (at 75.6285 31.75 0)
       (effects (font (size 1.27 1.27) italic) (justify left))
     )
@@
       )
     )
+  )
+  (sheet (at 24.13 92.71) (size 35.56 29.21) (fields_autoplaced)
+    (stroke (width 0.1524) (type solid))
+    (fill (color 0 0 0 0.0000))
+    (property "Sheetname" "Connector" (at 24.13 91.9984 0)
+      (effects (font (size 1.27 1.27)) (justify left bottom))
+    )
+    (property "Sheetfile" "connector.kicad_sch" (at 24.13 122.5046 0)
+      (effects (font (size 1.27 1.27)) (justify left top))
+    )
+    (instances
+      (project "pcb_redesign"
+        (path "/fb030e39-7dd3-46a0-8379-c26b3ef1b0a0" (page "2"))
+      )
+    )
