File: pcb_redesign/pcb_redesign.kicad_sch (KiCad schematic)
At the start: 6 parts, among them U1 ESP32-S3-WROOM-1

Commit message: Finished 1st draft of schematic
Connections:
- net D-: now reaches U1.13 (GPIO19/U1RTS/ADC2_CH8/CLK_OUT2/USB_D-)
- net D+: now reaches U1.14 (GPIO20/U1CTS/ADC2_CH9/CLK_OUT1/USB_D+)
- net ENB Right Motor: now reaches U1.38 (GPIO2/TOUCH2/ADC1_CH1)
- net ENA Right Motor: now reaches U1.39 (GPIO1/TOUCH1/ADC1_CH0)
- net ENA Left Motor: now reaches U1.4 (GPIO4/TOUCH4/ADC1_CH3)
- net ENB Left Motor: now reaches U1.5 (GPIO5/TOUCH5/ADC1_CH4)
- no-connect marks 0 -> 30
Other:
- added sheet Connector (connector.kicad_sch)
- added sheet motors (motors.kicad_sch)
- note added: "Goes to pad (and then gnd..?)"
- note added: "If I dont want a pin to be accessible, do I ground the pin or do I mark it as not connected"
- note added: "Note that GPIO 0 is default high unless connected otherwise, GPIO 45 default low, GPIO 46 default low"
- note added: "Seem to be missing epad and epad gnd, is this problem????"
