File: pcb_redesign/_autosave-connector.kicad_sch (KiCad schematic)
At the start: 8 parts, among them IC1 SPX1117M3-L-3-3_TR, J2 USB_B

Commit message: finished design
Parts:
- C4: footprint 1uF_cap_0603:CL10A105KB8NNNC -> Capacitor_SMD:C_0603_1608Metric
- IC1: footprint SOT230P700X180-4N -> 3.3v_reg:SOT230P700X180-4N
Changed lines of the file:
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@@
       (effects (font (size 1.27 1.27)) (justify left))
     )
-    (property "Footprint" "1uF_cap_0603:CL10A105KB8NNNC" (at 102.87 48.26 0)
+    (property "Footprint" "Capacitor_SMD:C_0603_1608Metric" (at 102.87 48.26 0)
       (effects (font (size 1.27 1.27)) hide)
     )
@@
       (effects (font (size 1.27 1.27)))
     )
-    (property "Footprint" "SOT230P700X180-4N" (at 168.91 49.53 0)
+    (property "Footprint" "3.3v_reg:SOT230P700X180-4N" (at 168.91 49.53 0)
       (effects (font (size 1.27 1.27)) (justify left) hide)
     )
